File: noname.kicad_pcb (KiCad board)
At the start: 2 copper layers, 41 parts, among them J1 JST, J2 ANEMOMETER, J3 USB_B_Micro, J4 Expansion, J5 SWD_PROG, J6 microSD, J8 Antenna, SW1 SW_DPDT_x2, U1 MCP73831-2-OT, U2 AP2112K-3.3, U3 W25Q64JVSSIM, U4 ATSAMD21G18A-AUT, U5 RFM95W-915S2, U6 BMP388, Y1 32.768 Hz

Commit message: 0 unrouted!
Parts:
- removed R7: 10k, footprints:R_0603_1608Metric
- moved C2 9.04 mm to (155.8, 161.2)
- moved R10 4.26 mm to (159.5, 158.5), turned to 180 degrees
- moved J8 3.13 mm to (130.2, 165.0)
- moved C6 2.69 mm to (158.8, 156.5), turned to 180 degrees
- moved U6 2.30 mm to (163.0, 156.8), turned to 270 degrees
- moved J6 1.90 mm to (140.8, 170.8), turned to 0 degrees
- moved J1 1.50 mm to (154.5, 170.5)
- moved C3 1.49 mm to (163.5, 161.2), turned to 180 degrees
- moved R5 1.27 mm to (161.2, 175.0)
- moved D1 1.25 mm to (161.3, 169.8), turned to 180 degrees
- moved D4 1.25 mm to (161.2, 172.5)
- moved C1 0.99 mm to (159.5, 161.2)
- moved R6 0.83 mm to (163.5, 166.2)
- moved U1 0.79 mm to (152.8, 165.5)
- moved U2 0.79 mm to (158.8, 165.5)
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Routing:
- net +3V3: track 23.4 -> 212.8 mm, vias 2 -> 11
- net GND: track 30.5 -> 130.4 mm, vias 6 -> 19
- net VBUS: track 1.77 -> 57.4 mm, vias 1 -> 3
- net /LORA_MISO: track 0.00 -> 25.6 mm, vias 0 -> 2
- net /microSD_CS: track 0.00 -> 25.3 mm, vias 0 -> 2
- net +BATT: track 0.00 -> 22.8 mm
- net /microSD_MOSI: track 0.00 -> 22.3 mm
- net /microSD_SCK: track 0.00 -> 21.3 mm
- net /microSD_MISO: track 0.00 -> 19.2 mm
- net Net-(R5-Pad2): track 0.00 -> 18.6 mm
- net /BATT_V: track 1.56 -> 18.6 mm, vias 1 -> 2
- net /BMP388_CS: track 0.00 -> 11.5 mm, vias 0 -> 2
- net Net-(SW1-Pad1): track 0.00 -> 7.21 mm
- net /BMP388_MISO: track 0.00 -> 6.48 mm, vias 0 -> 2
- net Net-(J8-Pad1): track 0.00 -> 6.21 mm
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- added copper zone on B.Cu, net GND
Other:
- board outline added: 44.5 x 42.2 mm

Commit message: Added labels
Routing:
- net GND: track 130.4 -> 129.0 mm
Other:
- board text added: "3V3"
- board text added: "ANEM"
- board text added: "ANT"
- board text added: "GND"
- board text added: "Hummingbird rev 1"
- board text added: "I2C SCL"
- board text added: "I2C SDA"
- board text added: "RESET"
- board text added: "RX"
- board text added: "SWCLK"
- board text added: "SWDIO"
- board text added: "TAHNOK"
- board text added: "TX"
Changed lines of the file:
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@@
   (general
     (thickness 1.6)
-    (drawings 6)
-    (tracks 590)
+    (drawings 23)
+    (tracks 592)
     (zones 0)
     (modules 40)
@@
     (at 140.75 170.75)
     (attr smd)
-    (fp_text reference J6 (at -8.64903 4.21685 90) (layer F.SilkS)
+    (fp_text reference J6 (at -0.25 0 90) (layer F.SilkS)
       (effects (font (size 1.00162 1.00162) (thickness 0.05)))
     )
@@
     (tags "test point SMD pad")
     (attr virtual)
-    (fp_text reference TP1 (at 0 1.448) (layer B.SilkS)
+    (fp_text reference TP1 (at 2.5 0) (layer B.SilkS)
       (effects (font (size 1 1) (thickness 0.15)) (justify mirror))
     )
@@
     (tags "test point SMD pad")
     (attr virtual)
-    (fp_text reference TP2 (at 0 1.448) (layer B.SilkS)
+    (fp_text reference TP2 (at 2.5 0) (layer B.SilkS)
       (effects (font (size 1 1) (thickness 0.15)) (justify mirror))
     )
@@
       (rotate (xyz 0 0 0))
     )
+  )
+  (gr_text "Hummingbird\nrev 1" (at 130.75 172.25 90) (layer F.SilkS)
+    (effects (font (size 1 1) (thickness 0.15)))
+  )
+  (gr_text TAHNOK (at 135 174.25 180) (layer B.Cu)
+    (effects (font (size 2 2) (thickness 0.5) italic) (justify mirror))
+  )
+  (gr_text ANT (at 130.25 169 90) (layer B.SilkS)
+    (effects (font (size 1.5 1.5) (thickness 0.3)) (justify mirror))
+  )
+  (gr_text ANEM (at 132 143 90) (layer B.SilkS)
+    (effects (font (size 1.5 1.5) (thickness 0.3)) (justify mirror))
+  )
+  (gr_text "I2C SDA" (at 142.25 144.25 90) (layer B.SilkS)
+    (effects (font (size 1.5 1.5) (thickness 0.3)) (justify mirror))
+  )
+  (gr_text "I2C SCL" (at 145.25 144.25 90) (layer B.SilkS)
+    (effects (font (size 1.5 1.5) (thickness 0.3)) (justify mirror))
+  )
+  (gr_text RX (at 147.75 141.25 90) (layer B.SilkS)
+    (effects (font (size 1.5 1.5) (thickness 0.3)) (justify mirror))
+  )
+  (gr_text TX (at 150.25 141.25 90) (layer B.SilkS)
+    (effects (font (size 1.5 1.5) (thickness 0.3)) (justify mirror))
+  )
+  (gr_text 3V3 (at 134.75 142 90) (layer B.SilkS)
+    (effects (font (size 1.5 1.5) (thickness 0.3)) (justify mirror))
+  )
+  (gr_text 3V3 (at 152.75 142 90) (layer B.SilkS)
+    (effects (font (size 1.5 1.5) (thickness 0.3)) (justify mirror))
+  )
+  (gr_text GND (at 137.25 142 90) (layer B.SilkS)
+    (effects (font (size 1.5 1.5) (thickness 0.3)) (justify mirror))
+  )
+  (gr_text GND (at 155.25 142 90) (layer B.SilkS)
+    (effects (font (size 1.5 1.5) (thickness 0.3)) (justify mirror))
+  )
+  (gr_text SWCLK (at 160.5 143.25 90) (layer B.SilkS)
+    (effects (font (size 1.5 1.5) (thickness 0.3)) (justify mirror))
+  )
+  (gr_text SWDIO (at 163.25 143 90) (layer B.SilkS)
+    (effects (font (size 1.5 1.5) (thickness 0.3)) (justify mirror))
+  )
+  (gr_text RESET (at 165.75 143 90) (layer B.SilkS)
+    (effects (font (size 1.5 1.5) (thickness 0.3)) (justify mirror))
+  )
+  (gr_text 3V3 (at 168.25 141.75 90) (layer B.SilkS)
+    (effects (font (size 1.5 1.5) (thickness 0.3)) (justify mirror))
+  )
+  (gr_text GND (at 170.75 142 90) (layer B.SilkS)
+    (effects (font (size 1.5 1.5) (thickness 0.3)) (justify mirror))
   )
   (gr_line (start 128.25 178.5) (end 128.25 136.25) (layer Edge.Cuts) (width 0.1))
@@
   (segment (start 152.75 160.062501) (end 151.2125 158.525001) (width 0.5) (layer F.Cu) (net 1))
   (segment (start 152.75 161.25) (end 152.75 160.062501) (width 0.5) (layer F.Cu) (net 1))
-  (segment (start 137.25 139.85) (end 137.25 138.5) (width 0.5) (layer F.Cu) (net 1))
-  (segment (start 136.450001 140.649999) (end 137.25 139.85) (width 0.5) (layer F.Cu) (net 1))
-  (segment (start 129.7523 143.10149) (end 132.203791 140.649999) (width 0.5) (layer F.Cu) (net 1))
   (segment (start 129.7523 144.00192) (end 129.7523 143.10149) (width 0.5) (layer F.Cu) (net 1))
   (segment (start 147.2125 143.25) (end 146 143.25) (width 0.5) (layer F.Cu) (net 1))
@@
   (segment (start 143.35 164.395) (end 143.35 163.4) (width 0.5) (layer F.Cu) (net 1))
   (segment (start 143.35 163.4) (end 143.5 163.25) (width 0.5) (layer F.Cu) (net 1))
-  (via (at 129.75 141.75) (size 0.8) (drill 0.4) (layers F.Cu B.Cu) (net 1))
-  (segment (start 129.7523 144.00192) (end 129.7523 141.7523) (width 0.5) (layer F.Cu) (net 1))
-  (segment (start 129.7523 141.7523) (end 129.75 141.75) (width 0.5) (layer F.Cu) (net 1))
   (segment (start 167.595 158.15) (end 167.595 157.845) (width 0.5) (layer F.Cu) (net 1))
   (segment (start 167.595 158.15) (end 166.849798 158.895202) (width 0.5) (layer F.Cu) (net 1))
@@
   (segment (start 161.5 161.25) (end 162.75 161.25) (width 0.5) (layer F.Cu) (net 1))
   (via (at 134.25 141) (size 0.8) (drill 0.4) (layers F.Cu B.Cu) (net 1))
-  (segment (start 134 140.75) (end 134.25 141) (width 0.5) (layer F.Cu) (net 1))
-  (segment (start 134 140.649999) (end 134 140.75) (width 0.5) (layer F.Cu) (net 1))
-  (segment (start 134 140.649999) (end 136.450001 140.649999) (width 0.5) (layer F.Cu) (net 1))
-  (segment (start 132.203791 140.649999) (end 134 140.649999) (width 0.5) (layer F.Cu) (net 1))
   (segment (start 163.113388 141.288388) (end 163.575 141.75) (width 0.5) (layer F.Cu) (net 1))
   (segment (start 161.625001 139.800001) (end 163.113388 141.288388) (width 0.5) (layer F.Cu) (net 1))
@@
   (segment (start 143.75 141.75) (end 148.33326 141.75) (width 1) (layer F.Cu) (net 1))
   (via (at 148.33326 141.75) (size 0.8) (drill 0.4) (layers F.Cu B.Cu) (net 1))
+  (via (at 129.75 141.75) (size 0.8) (drill 0.4) (layers F.Cu B.Cu) (net 1))
+  (segment (start 129.7523 144.00192) (end 129.7523 141.7523) (width 1) (layer F.Cu) (net 1))
+  (segment (start 129.7523 141.7523) (end 129.75 141.75) (width 1) (layer F.Cu) (net 1))
+  (segment (start 129.75 141.75) (end 129.75 141) (width 1) (layer F.Cu) (net 1))
+  (segment (start 129.75 141) (end 134.25 141) (width 1) (layer F.Cu) (net 1))
+  (segment (start 137.004002 138.5) (end 137.25 138.5) (width 1) (layer F.Cu) (net 1))
+  (segment (start 134.904001 140.600001) (end 137.004002 138.5) (width 1) (layer F.Cu) (net 1))
+  (segment (start 134.649999 140.600001) (end 134.904001 140.600001) (width 1) (layer F.Cu) (net 1))
+  (segment (start 134.25 141) (end 134.649999 140.600001) (width 1) (layer F.Cu) (net 1))
   (segment (start 162.0375 169.7875) (end 162.075 169.75) (width 0.5) (layer F.Cu) (net 2))
   (segment (start 162.0375 172.5) (end 162.0375 169.7875) (width 0.5) (layer F.Cu) (net 2))
@@
   (segment (start 158.675 165.190002) (end 158.675 162.75) (width 0.5) (layer F.Cu) (net 2))
   (segment (start 168.47499 143.77501) (end 168.5 143.75) (width 0.5) (layer F.Cu) (net 2))
-  (segment (start 168.47499 150.00001) (end 168.47499 143.77501) (width 1) (layer F.Cu) (net 2))
   (segment (start 168.175 150.3) (end 168.47499 150.00001) (width 0.5) (layer F.Cu) (net 2))
   (segment (start 167 150.3) (end 168.175 150.3) (width 0.5) (layer F.Cu) (net 2))
@@
   (segment (start 161.258002 162.75) (end 166.92499 157.083012) (width 1) (layer B.Cu) (net 2))
   (segment (start 154.315685 162.75) (end 161.258002 162.75) (width 1) (layer B.Cu) (net 2))
+  (segment (start 168.17501 144.168728) (end 168.493729 143.850009) (width 1) (layer F.Cu) (net 2))
+  (segment (start 168.17501 146.92501) (end 168.17501 144.168728) (width 1) (layer F.Cu) (net 2))
+  (segment (start 168.47499 147.22499) (end 168.17501 146.92501) (width 1) (layer F.Cu) (net 2))
+  (segment (start 168.47499 150.00001) (end 168.47499 147.22499) (width 1) (layer F.Cu) (net 2))
   (segment (start 155.5 170.5) (end 155.5 168.4) (width 0.5) (layer F.Cu) (net 3))
   (segment (start 155.5 168.4) (end 155.5 163.5) (width 0.5) (layer F.Cu) (net 3))
@@
   (segment (start 152 151.568994) (end 151.568994 152) (width 0.25) (layer F.Cu) (net 59))
   (segment (start 129.7523 164.5023) (end 130.25 165) (width 0.5) (layer F.Cu) (net 67))
-  (segment (start 129.7523 158.99808) (end 129.7523 164.5023) (width 0.5) (layer F.Cu) (net 67))
+  (segment (start 129.7523 158.99808) (end 129.7523 164.5023) (width 1) (layer F.Cu) (net 67))
   (zone (net 1) (net_name GND) (layer B.Cu) (hatch edge 0.508)
     (connect_pads (clearance 0.508))

Commit message: add hummingbird drawing
Parts:
- added REF**: hummingbird, footprints:hummingbird, B.Cu at (154.0, 173.8)
